Commit message: Week4

File: Ros2_WS/install/robot_description/share/robot_description/urdf/fishbot/actuator/caster.urdf.xacro (robot description, xacro)
@@ -29,4 +29,10 @@
             <origin xyz="${xyz}" rpy="0.0 0.0 0.0"/>
         </joint>
+        <gazebo reference="${caster_name}_link">
+            <mu1 value="0.0"/>
+            <mu2 value="0.0"/>
+            <kp value="1000000000.0"/>
+            <kd value="1.0"/>
+        </gazebo>
     </xacro:macro>
 </robot>

File: Ros2_WS/install/robot_description/share/robot_description/urdf/fishbot/actuator/wheel.urdf.xacro (robot description, xacro)
@@ -30,4 +30,10 @@
             <axis xyz="0 1 0"/>
         </joint>
+        <gazebo reference="${wheel_name}_link">
+            <mu1 value="20.0"/>
+            <mu2 value="20.0"/>
+            <kp value="1000000000.0"/>
+            <kd value="1.0"/>
+        </gazebo>
     </xacro:macro>
 </robot>

File: Ros2_WS/install/robot_description/share/robot_description/urdf/fishbot/fishbot.urdf.xacro (robot description, xacro)
@@ -7,4 +7,6 @@
 <xacro:include filename="$(find robot_description)/urdf/fishbot/actuator/wheel.urdf.xacro"/>
 <xacro:include filename="$(find robot_description)/urdf/fishbot/actuator/caster.urdf.xacro"/>
+<xacro:include filename="$(find robot_description)/urdf/fishbot/plugins/gazebo_control_plugin.xacro"/>
+<xacro:include filename="$(find robot_description)/urdf/fishbot/plugins/gazebo_sensor_plugin.xacro"/>
 <xacro:base_xacro length="0.12" radius="0.10"/>
 <xacro:imu_xacro xyz="0.0 0.0 0.0"/>
@@ -15,3 +17,5 @@
 <xacro:caster_xacro caster_name="front_wheel" xyz="0.08 0.0 -0.076"/>
 <xacro:caster_xacro caster_name="back_wheel" xyz="-0.08 0.0 -0.076"/>
+<xacro:gazebo_control_plugin/>
+<xacro:gazebo_sensor_plugin/>
 </robot>

File: Ros2_WS/install/robot_description/share/robot_description/urdf/fishbot/sensor/camera.urdf.xacro (robot description, xacro)
@@ -24,4 +24,5 @@
             <xacro:box_inertia m="0.10" w="0.02" h="0.10" d="0.02"/>
         </link>
+        <link name="camera_optical_link" />
         <joint name="camera_joint" type="fixed">
             <parent link="base_link"/>
@@ -29,4 +30,9 @@
             <origin xyz="${xyz}" rpy="0.0 0.0 0.0"/>
         </joint>
+        <joint name="camera_optical_joint" type="fixed">
+            <parent link="camera_link"/>
+            <child link="camera_optical_link"/>
+            <origin xyz="0 0 0" rpy="${-pi/2} 0.0 ${-pi/2}"/>
+        </joint>
     </xacro:macro>
 </robot>

File: Ros2_WS/install/robot_description/share/robot_description/urdf/fishbot/sensor/laser.urdf.xacro (robot description, xacro)
@@ -55,4 +55,10 @@
             <origin xyz="0.0 0.0 0.05" rpy="0.0 0.0 0.0"/>
         </joint>
+        <gazebo reference="laser_cylinder_link">
+            <material>Gazebo/Black</material>
+        </gazebo>
+        <gazebo reference="laser_link">
+            <material>Gazebo/Black</material>
+        </gazebo>
     </xacro:macro>
 </robot>
